File: pcb/megashield_svn_1.3_geoeffnet/Batteriespannung.sch (KiCad schematic (older format))
At the start: 4 parts

Commit message: Import dernière version
1.0a4-Azurit
Parts:
- removed CC5: 100nF, Capacitors_ThroughHole:C_Disc_D3_P2.5, symbol Kondensator
Changed lines of the file:
@@
 EESchema Schematic File Version 2
+LIBS:ardumower mega shield svn-cache
 LIBS:Wlan_ESP8266
 LIBS:power
-LIBS:ardumower mega shield svn-cache
+LIBS:conn
+LIBS:uln-udn
 EELAYER 25 0
 EELAYER END
@@
 	6340 1755 6340 1970
 $Comp
-L GND #PWR0172
+L GND #PWR0180
 U 1 1 554BD908
 P 6340 2600
-F 0 "#PWR0172" H 6340 2350 60  0001 C CNN
+F 0 "#PWR0180" H 6340 2350 60  0001 C CNN
 F 1 "GND" H 6340 2450 60  0000 C CNN
 F 2 "" H 6340 2600 60  0000 C CNN
@@
 	6340 2470 6340 2600
 $Comp
-L GND #PWR0173
+L GND #PWR0181
 U 1 1 554C8CE9
 P 6660 2600
-F 0 "#PWR0173" H 6660 2350 60  0001 C CNN
+F 0 "#PWR0181" H 6660 2350 60  0001 C CNN
 F 1 "GND" H 6660 2450 60  0000 C CNN
 F 2 "" H 6660 2600 60  0000 C CNN
@@
 Wire Wire Line
 	6660 1870 6660 1995
-Wire Wire Line
-	5885 1870 6900 1870
 Connection ~ 6340 1870
 Text HLabel 5475 1150 0    60   Input ~ 0
@@
 pinBatteryVoltage
 Connection ~ 6660 1870
-$Comp
-L Kondensator CC5
-U 1 1 5558A3B2
-P 5885 2215
-F 0 "CC5" H 5935 2315 50  0000 L CNN
-F 1 "100nF" H 5935 2115 50  0000 L CNN
-F 2 "Capacitors_ThroughHole:C_Disc_D3_P2.5" H 5885 2215 60  0001 C CNN
-F 3 "" H 5885 2215 60  0000 C CNN
-F 4 "R: KERKO 100N" H 5885 2215 60  0001 C CNN "Bestellnummer"
-F 5 "http://www.reichelt.de/Scheiben/KERKO-100N/3/index.html?&ACTION=3&LA=2&ARTICLE=9265&GROUPID=3169&artnr=KERKO+100N" H 5885 2215 60  0001 C CNN "Bestelllink"
-	1    5885 2215
-	1    0    0    -1
-$EndComp
-$Comp
-L GND #PWR0174
-U 1 1 5558A47F
-P 5885 2600
-F 0 "#PWR0174" H 5885 2350 60  0001 C CNN
-F 1 "GND" H 5885 2450 60  0000 C CNN
-F 2 "" H 5885 2600 60  0000 C CNN
-F 3 "" H 5885 2600 60  0000 C CNN
-	1    5885 2600
-	1    0    0    -1
-$EndComp
 Wire Wire Line
-	5885 2600 5885 2415
-Wire Wire Line
-	5885 1870 5885 2015
+	6900 1870 6340 1870
 $EndSCHEMATC
