File: pcb/megashield_svn_1.3_geoeffnet/Dual1_Ms_Links.sch (KiCad schematic (older format))
At the start: 7 parts, among them P18 Left

Commit message: Import dernière version
1.0a4-Azurit
Changed lines of the file:
@@
 EESchema Schematic File Version 2
+LIBS:ardumower mega shield svn-cache
 LIBS:Wlan_ESP8266
 LIBS:power
-LIBS:ardumower mega shield svn-cache
+LIBS:conn
+LIBS:uln-udn
 EELAYER 25 0
 EELAYER END
@@
 P 4895 3310
 AR Path="/553D8AD9/5542A35A/554BE910" Ref="#PWR0137"  Part="1"
-AR Path="/553D8AD9/554D3EE8/554BE910" Ref="#PWR0143"  Part="1"
-F 0 "#PWR0143" H 4895 3160 60  0001 C CNN
+AR Path="/553D8AD9/554D3EE8/554BE910" Ref="#PWR0149"  Part="1"
+F 0 "#PWR0149" H 4895 3160 60  0001 C CNN
 F 1 "+24V" H 4895 3450 60  0000 C CNN
 F 2 "" H 4895 3310 60  0000 C CNN
@@
 P 4895 4445
 AR Path="/553D8AD9/5542A35A/5542A3C5" Ref="#PWR0138"  Part="1"
-AR Path="/553D8AD9/554D3EE8/5542A3C5" Ref="#PWR0144"  Part="1"
-F 0 "#PWR0144" H 4895 4195 60  0001 C CNN
+AR Path="/553D8AD9/554D3EE8/5542A3C5" Ref="#PWR0150"  Part="1"
+F 0 "#PWR0150" H 4895 4195 60  0001 C CNN
 F 1 "GND" H 4895 4295 60  0000 C CNN
 F 2 "" H 4895 4445 60  0000 C CNN
@@
 P 4895 3580
 AR Path="/553D8AD9/5542A35A/5542A3D9" Ref="BY3"  Part="1"
-AR Path="/553D8AD9/554D3EE8/5542A3D9" Ref="BY7"  Part="1"
-F 0 "BY7" H 4895 3680 40  0000 C CNN
+AR Path="/553D8AD9/554D3EE8/5542A3D9" Ref="DBY7"  Part="1"
+F 0 "DBY7" H 4895 3680 40  0000 C CNN
 F 1 "BY 500/1000" H 4895 3480 40  0000 C CNN
 F 2 "ACS712:Diode_liegend_BY500_1000_RM10" H 4895 3580 60  0001 C CNN
@@
 P 4895 4140
 AR Path="/553D8AD9/5542A35A/5542A4FC" Ref="BY4"  Part="1"
-AR Path="/553D8AD9/554D3EE8/5542A4FC" Ref="BY8"  Part="1"
-F 0 "BY8" H 4895 4240 40  0000 C CNN
+AR Path="/553D8AD9/554D3EE8/5542A4FC" Ref="DBY8"  Part="1"
+F 0 "DBY8" H 4895 4240 40  0000 C CNN
 F 1 "BY 500/1000" H 4895 4040 40  0000 C CNN
 F 2 "ACS712:Diode_liegend_BY500_1000_RM10" H 4895 4140 60  0001 C CNN
@@
 P 3170 3310
 AR Path="/553D8AD9/5542A35A/5542A69A" Ref="#PWR0139"  Part="1"
-AR Path="/553D8AD9/554D3EE8/5542A69A" Ref="#PWR0145"  Part="1"
-F 0 "#PWR0145" H 3170 3160 60  0001 C CNN
+AR Path="/553D8AD9/554D3EE8/5542A69A" Ref="#PWR0151"  Part="1"
+F 0 "#PWR0151" H 3170 3160 60  0001 C CNN
 F 1 "+24V" H 3170 3450 60  0000 C CNN
 F 2 "" H 3170 3310 60  0000 C CNN
@@
 P 3170 4445
 AR Path="/553D8AD9/5542A35A/554BE919" Ref="#PWR0140"  Part="1"
-AR Path="/553D8AD9/554D3EE8/554BE919" Ref="#PWR0146"  Part="1"
-F 0 "#PWR0146" H 3170 4195 60  0001 C CNN
+AR Path="/553D8AD9/554D3EE8/554BE919" Ref="#PWR0152"  Part="1"
+F 0 "#PWR0152" H 3170 4195 60  0001 C CNN
 F 1 "GND" H 3170 4295 60  0000 C CNN
 F 2 "" H 3170 4445 60  0000 C CNN
@@
 P 3170 3580
 AR Path="/553D8AD9/5542A35A/554BE91B" Ref="BY1"  Part="1"
-AR Path="/553D8AD9/554D3EE8/554BE91B" Ref="BY5"  Part="1"
-F 0 "BY5" H 3170 3680 40  0000 C CNN
+AR Path="/553D8AD9/554D3EE8/554BE91B" Ref="DBY5"  Part="1"
+F 0 "DBY5" H 3170 3680 40  0000 C CNN
 F 1 "BY 500/1000" H 3170 3480 40  0000 C CNN
 F 2 "ACS712:Diode_liegend_BY500_1000_RM10" H 3170 3580 60  0001 C CNN
@@
 P 3170 4140
 AR Path="/553D8AD9/5542A35A/554BE91D" Ref="BY2"  Part="1"
-AR Path="/553D8AD9/554D3EE8/554BE91D" Ref="BY6"  Part="1"
-F 0 "BY6" H 3170 4240 40  0000 C CNN
+AR Path="/553D8AD9/554D3EE8/554BE91D" Ref="DBY6"  Part="1"
+F 0 "DBY6" H 3170 4240 40  0000 C CNN
 F 1 "BY 500/1000" H 3170 4040 40  0000 C CNN
 F 2 "ACS712:Diode_liegend_BY500_1000_RM10" H 3170 4140 60  0001 C CNN
