File: pcb/megashield_svn_1.3_geoeffnet/Dual1_Ms_Rechts.sch (KiCad schematic (older format))
At the start: 7 parts, among them P18 Right

Commit message: Import dernière version
1.0a4-Azurit
Parts:
- renumbered BY1 to DBY1, BY2 to DBY2, BY3 to DBY3, BY4 to DBY4
Changed lines of the file:
@@
 EESchema Schematic File Version 2
+LIBS:ardumower mega shield svn-cache
 LIBS:Wlan_ESP8266
 LIBS:power
-LIBS:ardumower mega shield svn-cache
+LIBS:conn
+LIBS:uln-udn
 EELAYER 25 0
 EELAYER END
@@
 MotorRechtsB
 $Comp
-L +24V #PWR0137
+L +24V #PWR0143
 U 1 1 554BE90F
 P 4895 3310
-F 0 "#PWR0137" H 4895 3160 60  0001 C CNN
+F 0 "#PWR0143" H 4895 3160 60  0001 C CNN
 F 1 "+24V" H 4895 3450 60  0000 C CNN
 F 2 "" H 4895 3310 60  0000 C CNN
@@
 $EndComp
 $Comp
-L GND #PWR0138
+L GND #PWR0144
 U 1 1 554BE911
 P 4895 4445
-F 0 "#PWR0138" H 4895 4195 60  0001 C CNN
+F 0 "#PWR0144" H 4895 4195 60  0001 C CNN
 F 1 "GND" H 4895 4295 60  0000 C CNN
 F 2 "" H 4895 4445 60  0000 C CNN
@@
 $EndComp
 $Comp
-L DIODE BY3
+L DIODE DBY3
 U 1 1 554BE913
 P 4895 3580
-F 0 "BY3" H 4895 3680 40  0000 C CNN
+F 0 "DBY3" H 4895 3680 40  0000 C CNN
 F 1 "BY 500/1000" H 4895 3480 40  0000 C CNN
 F 2 "ACS712:Diode_liegend_BY500_1000_RM15" H 4895 3580 60  0001 C CNN
@@
 $EndComp
 $Comp
-L DIODE BY4
+L DIODE DBY4
 U 1 1 554BE915
 P 4895 4140
-F 0 "BY4" H 4895 4240 40  0000 C CNN
+F 0 "DBY4" H 4895 4240 40  0000 C CNN
 F 1 "BY 500/1000" H 4895 4040 40  0000 C CNN
 F 2 "ACS712:Diode_liegend_BY500_1000_RM15" H 4895 4140 60  0001 C CNN
@@
 Connection ~ 4895 3870
 $Comp
-L +24V #PWR0139
+L +24V #PWR0145
 U 1 1 554BE918
 P 3170 3310
-F 0 "#PWR0139" H 3170 3160 60  0001 C CNN
+F 0 "#PWR0145" H 3170 3160 60  0001 C CNN
 F 1 "+24V" H 3170 3450 60  0000 C CNN
 F 2 "" H 3170 3310 60  0000 C CNN
@@
 $EndComp
 $Comp
-L GND #PWR0140
+L GND #PWR0146
 U 1 1 554BE91A
 P 3170 4445
-F 0 "#PWR0140" H 3170 4195 60  0001 C CNN
+F 0 "#PWR0146" H 3170 4195 60  0001 C CNN
 F 1 "GND" H 3170 4295 60  0000 C CNN
 F 2 "" H 3170 4445 60  0000 C CNN
@@
 $EndComp
 $Comp
-L DIODE BY1
+L DIODE DBY1
 U 1 1 554BE91C
 P 3170 3580
-F 0 "BY1" H 3170 3680 40  0000 C CNN
+F 0 "DBY1" H 3170 3680 40  0000 C CNN
 F 1 "BY 500/1000" H 3170 3480 40  0000 C CNN
 F 2 "ACS712:Diode_liegend_BY500_1000_RM15" H 3170 3580 60  0001 C CNN
@@
 $EndComp
 $Comp
-L DIODE BY2
+L DIODE DBY2
 U 1 1 554BE91E
 P 3170 4140
-F 0 "BY2" H 3170 4240 40  0000 C CNN
+F 0 "DBY2" H 3170 4240 40  0000 C CNN
 F 1 "BY 500/1000" H 3170 4040 40  0000 C CNN
 F 2 "ACS712:Diode_liegend_BY500_1000_RM15" H 3170 4140 60  0001 C CNN
