File: pcb/megashield_svn_1.3_geoeffnet/Dual1_Vin.sch (KiCad schematic (older format))
At the start: 3 parts, among them P16 V.OUT

Commit message: Import dernière version
1.0a4-Azurit
Parts:
- added C12: 2200uF 63V, symbol CP1
- renumbered KE3 to DKE3
Connections:
- net Dual1_Vin: now also C12.1
- net GND: now also C12.2
Changed lines of the file:
@@
 EESchema Schematic File Version 2
+LIBS:ardumower mega shield svn-cache
 LIBS:Wlan_ESP8266
 LIBS:power
-LIBS:ardumower mega shield svn-cache
+LIBS:conn
+LIBS:uln-udn
 EELAYER 25 0
 EELAYER END
@@
 $EndComp
 $Comp
-L +24V #PWR0141
+L +24V #PWR0147
 U 1 1 5543AA9F
 P 4370 2960
-F 0 "#PWR0141" H 4370 2810 60  0001 C CNN
+F 0 "#PWR0147" H 4370 2810 60  0001 C CNN
 F 1 "+24V" H 4370 3100 60  0000 C CNN
 F 2 "" H 4370 2960 60  0000 C CNN
@@
 $EndComp
 $Comp
-L GND #PWR0142
+L GND #PWR0148
 U 1 1 554BE925
 P 4370 4555
-F 0 "#PWR0142" H 4370 4305 60  0001 C CNN
+F 0 "#PWR0148" H 4370 4305 60  0001 C CNN
 F 1 "GND" H 4370 4405 60  0000 C CNN
 F 2 "" H 4370 4555 60  0000 C CNN
@@
 	1    0    0    -1
 $EndComp
-Text HLabel 4030 3700 0    60   Input ~ 0
+Text HLabel 3190 3700 0    60   Input ~ 0
 Dual1_Vin
-Text HLabel 4045 4290 0    60   Input ~ 0
+Text HLabel 3180 4290 0    60   Input ~ 0
 Dual1_GND
 Wire Wire Line
 	4370 3415 4370 3855
 Wire Wire Line
-	4370 4555 4370 4155
+	4370 4155 4370 4555
 $Comp
-L 15KEXXC KE3
+L 15KEXXC DKE3
 U 1 1 5543B245
 P 4370 3955
-F 0 "KE3" V 4440 4165 50  0000 L BNN
+F 0 "DKE3" V 4440 4165 50  0000 L BNN
 F 1 "15KE33CA" V 4520 4035 50  0000 L BNN
 F 2 "ACS712:Diode_15KE33CA" H 4370 4105 50  0001 C CNN
@@
 $EndComp
 Wire Wire Line
-	4030 3700 4640 3700
+	3190 3700 4640 3700
 Connection ~ 4370 3700
 Wire Wire Line
-	4045 4290 4640 4290
+	3180 4290 4640 4290
 Connection ~ 4370 4290
 Wire Wire Line
@@
 Wire Wire Line
 	4370 3015 4370 2960
+$Comp
+L CP1 C12
+U 1 1 55723D66
+P 3325 3990
+F 0 "C12" H 3375 4090 50  0000 L CNN
+F 1 "2200uF 63V" H 3375 3890 50  0000 L CNN
+F 2 "" H 3325 3990 60  0001 C CNN
+F 3 "" H 3325 3990 60  0000 C CNN
+F 4 "Value" H 3325 3990 60  0001 C CNN "Bestellnummer"
+F 5 "Value" H 3325 3990 60  0001 C CNN "Bestelllink"
+	1    3325 3990
+	1    0    0    -1
+$EndComp
+Wire Wire Line
+	3325 3790 3325 3700
+Connection ~ 3325 3700
+Wire Wire Line
+	3325 4190 3325 4290
+Connection ~ 3325 4290
 $EndSCHEMATC
