File: pcb/megashield_svn_1.3_geoeffnet/Dual2_Ms_Mower.sch (KiCad schematic (older format))
At the start: 7 parts, among them P18 Mower

Commit message: Import dernière version
1.0a4-Azurit
Changed lines of the file:
@@
 EESchema Schematic File Version 2
+LIBS:ardumower mega shield svn-cache
 LIBS:Wlan_ESP8266
 LIBS:power
-LIBS:ardumower mega shield svn-cache
+LIBS:conn
+LIBS:uln-udn
 EELAYER 25 0
 EELAYER END
@@
 AR Path="/553D8AD9/5542A35A/5542A3B1" Ref="#PWR0130"  Part="1"
 AR Path="/553D8AD9/554D3EE8/5542A3B1" Ref="#PWR0136"  Part="1"
-AR Path="/553D8AD9/554D4C79/5542A3B1" Ref="#PWR0147"  Part="1"
-F 0 "#PWR0147" H 4895 3160 60  0001 C CNN
+AR Path="/553D8AD9/554D4C79/5542A3B1" Ref="#PWR0153"  Part="1"
+F 0 "#PWR0153" H 4895 3160 60  0001 C CNN
 F 1 "+24V" H 4895 3450 60  0000 C CNN
 F 2 "" H 4895 3310 60  0000 C CNN
@@
 AR Path="/553D8AD9/5542A35A/554BE912" Ref="#PWR0131"  Part="1"
 AR Path="/553D8AD9/554D3EE8/554BE912" Ref="#PWR0137"  Part="1"
-AR Path="/553D8AD9/554D4C79/554BE912" Ref="#PWR0148"  Part="1"
-F 0 "#PWR0148" H 4895 4195 60  0001 C CNN
+AR Path="/553D8AD9/554D4C79/554BE912" Ref="#PWR0154"  Part="1"
+F 0 "#PWR0154" H 4895 4195 60  0001 C CNN
 F 1 "GND" H 4895 4295 60  0000 C CNN
 F 2 "" H 4895 4445 60  0000 C CNN
@@
 AR Path="/553D8AD9/5542A35A/554BE914" Ref="BY3"  Part="1"
 AR Path="/553D8AD9/554D3EE8/554BE914" Ref="BY7"  Part="1"
-AR Path="/553D8AD9/554D4C79/554BE914" Ref="BY11"  Part="1"
-F 0 "BY11" H 4895 3680 40  0000 C CNN
+AR Path="/553D8AD9/554D4C79/554BE914" Ref="DBY11"  Part="1"
+F 0 "DBY11" H 4895 3680 40  0000 C CNN
 F 1 "BY 500/1000" H 4895 3480 40  0000 C CNN
 F 2 "ACS712:Diode_liegend_BY500_1000_RM15" H 4895 3580 60  0001 C CNN
@@
 AR Path="/553D8AD9/5542A35A/554BE916" Ref="BY4"  Part="1"
 AR Path="/553D8AD9/554D3EE8/554BE916" Ref="BY8"  Part="1"
-AR Path="/553D8AD9/554D4C79/554BE916" Ref="BY12"  Part="1"
-F 0 "BY12" H 4895 4240 40  0000 C CNN
+AR Path="/553D8AD9/554D4C79/554BE916" Ref="DBY12"  Part="1"
+F 0 "DBY12" H 4895 4240 40  0000 C CNN
 F 1 "BY 500/1000" H 4895 4040 40  0000 C CNN
 F 2 "ACS712:Diode_liegend_BY500_1000_RM15" H 4895 4140 60  0001 C CNN
@@
 AR Path="/553D8AD9/5542A35A/554BE917" Ref="#PWR0132"  Part="1"
 AR Path="/553D8AD9/554D3EE8/554BE917" Ref="#PWR0138"  Part="1"
-AR Path="/553D8AD9/554D4C79/554BE917" Ref="#PWR0149"  Part="1"
-F 0 "#PWR0149" H 3170 3160 60  0001 C CNN
+AR Path="/553D8AD9/554D4C79/554BE917" Ref="#PWR0155"  Part="1"
+F 0 "#PWR0155" H 3170 3160 60  0001 C CNN
 F 1 "+24V" H 3170 3450 60  0000 C CNN
 F 2 "" H 3170 3310 60  0000 C CNN
@@
 AR Path="/553D8AD9/5542A35A/5542A6A0" Ref="#PWR0133"  Part="1"
 AR Path="/553D8AD9/554D3EE8/5542A6A0" Ref="#PWR0139"  Part="1"
-AR Path="/553D8AD9/554D4C79/5542A6A0" Ref="#PWR0150"  Part="1"
-F 0 "#PWR0150" H 3170 4195 60  0001 C CNN
+AR Path="/553D8AD9/554D4C79/5542A6A0" Ref="#PWR0156"  Part="1"
+F 0 "#PWR0156" H 3170 4195 60  0001 C CNN
 F 1 "GND" H 3170 4295 60  0000 C CNN
 F 2 "" H 3170 4445 60  0000 C CNN
@@
 AR Path="/553D8AD9/5542A35A/5542A6A6" Ref="BY1"  Part="1"
 AR Path="/553D8AD9/554D3EE8/5542A6A6" Ref="BY5"  Part="1"
-AR Path="/553D8AD9/554D4C79/5542A6A6" Ref="BY9"  Part="1"
-F 0 "BY9" H 3170 3680 40  0000 C CNN
+AR Path="/553D8AD9/554D4C79/5542A6A6" Ref="DBY9"  Part="1"
+F 0 "DBY9" H 3170 3680 40  0000 C CNN
 F 1 "BY 500/1000" H 3170 3480 40  0000 C CNN
 F 2 "ACS712:Diode_liegend_BY500_1000_RM15" H 3170 3580 60  0001 C CNN
@@
 AR Path="/553D8AD9/5542A35A/5542A6AC" Ref="BY2"  Part="1"
 AR Path="/553D8AD9/554D3EE8/5542A6AC" Ref="BY6"  Part="1"
-AR Path="/553D8AD9/554D4C79/5542A6AC" Ref="BY10"  Part="1"
-F 0 "BY10" H 3170 4240 40  0000 C CNN
+AR Path="/553D8AD9/554D4C79/5542A6AC" Ref="DBY10"  Part="1"
+F 0 "DBY10" H 3170 4240 40  0000 C CNN
 F 1 "BY 500/1000" H 3170 4040 40  0000 C CNN
 F 2 "ACS712:Diode_liegend_BY500_1000_RM15" H 3170 4140 60  0001 C CNN
