File: pcb/megashield_svn_1.3_geoeffnet/Dual2_Vin.sch (KiCad schematic (older format))
At the start: 3 parts, among them P16 V.OUT

Commit message: Import dernière version
1.0a4-Azurit
Parts:
- added C13: 2200uF 63V, symbol CP1
Connections:
- net Dual2_Vin: now also C13.1
- net GND: now also C13.2
Changed lines of the file:
@@
 EESchema Schematic File Version 2
+LIBS:ardumower mega shield svn-cache
 LIBS:Wlan_ESP8266
 LIBS:power
-LIBS:ardumower mega shield svn-cache
+LIBS:conn
+LIBS:uln-udn
 EELAYER 25 0
 EELAYER END
@@
 P 4370 2960
 AR Path="/553D8AD9/5543A988/554BE924" Ref="#PWR0134"  Part="1"
-AR Path="/553D8AD9/554D9DA2/554BE924" Ref="#PWR0151"  Part="1"
-F 0 "#PWR0151" H 4370 2810 60  0001 C CNN
+AR Path="/553D8AD9/554D9DA2/554BE924" Ref="#PWR0157"  Part="1"
+F 0 "#PWR0157" H 4370 2810 60  0001 C CNN
 F 1 "+24V" H 4370 3100 60  0000 C CNN
 F 2 "" H 4370 2960 60  0000 C CNN
@@
 P 4370 4555
 AR Path="/553D8AD9/5543A988/5543AAB4" Ref="#PWR0135"  Part="1"
-AR Path="/553D8AD9/554D9DA2/5543AAB4" Ref="#PWR0152"  Part="1"
-F 0 "#PWR0152" H 4370 4305 60  0001 C CNN
+AR Path="/553D8AD9/554D9DA2/5543AAB4" Ref="#PWR0158"  Part="1"
+F 0 "#PWR0158" H 4370 4305 60  0001 C CNN
 F 1 "GND" H 4370 4405 60  0000 C CNN
 F 2 "" H 4370 4555 60  0000 C CNN
@@
 	1    0    0    -1
 $EndComp
-Text HLabel 4030 3700 0    60   Input ~ 0
+Text HLabel 3130 3700 0    60   Input ~ 0
 Dual2_Vin
-Text HLabel 4045 4290 0    60   Input ~ 0
+Text HLabel 3130 4290 0    60   Input ~ 0
 Dual2_GND
 Wire Wire Line
 	4370 3415 4370 3855
 Wire Wire Line
-	4370 4555 4370 4155
+	4370 4155 4370 4555
 $Comp
 L 15KEXXC KE3
@@
 P 4370 3955
 AR Path="/553D8AD9/5543A988/554BE926" Ref="KE3"  Part="1"
-AR Path="/553D8AD9/554D9DA2/554BE926" Ref="KE4"  Part="1"
-F 0 "KE4" V 4440 4165 50  0000 L BNN
+AR Path="/553D8AD9/554D9DA2/554BE926" Ref="DKE4"  Part="1"
+F 0 "DKE4" V 4440 4165 50  0000 L BNN
 F 1 "15KE33CA" V 4520 4035 50  0000 L BNN
 F 2 "ACS712:Diode_15KE33CA" H 4370 4105 50  0001 C CNN
@@
 $EndComp
 Wire Wire Line
-	4030 3700 4640 3700
+	3130 3700 4640 3700
 Connection ~ 4370 3700
 Wire Wire Line
-	4045 4290 4640 4290
+	3130 4290 4640 4290
 Connection ~ 4370 4290
 Wire Wire Line
@@
 Wire Wire Line
 	4370 3015 4370 2960
+$Comp
+L CP1 C13
+U 1 1 55723BFA
+P 3350 3995
+F 0 "C13" H 3400 4095 50  0000 L CNN
+F 1 "2200uF 63V" H 3400 3895 50  0000 L CNN
+F 2 "" H 3350 3995 60  0001 C CNN
+F 3 "" H 3350 3995 60  0000 C CNN
+F 4 "Value" H 3350 3995 60  0001 C CNN "Bestellnummer"
+F 5 "Value" H 3350 3995 60  0001 C CNN "Bestelllink"
+	1    3350 3995
+	1    0    0    -1
+$EndComp
+Wire Wire Line
+	3350 3795 3350 3700
+Connection ~ 3350 3700
+Wire Wire Line
+	3350 4195 3350 4290
+Connection ~ 3350 4290
 $EndSCHEMATC
