File: pcb/megashield_svn_1.3_geoeffnet/Motortreiber.sch (KiCad schematic (older format))
At the start: 9 parts, among them P36 Res24V-2, P39 Res24V-1

Commit message: Import dernière version
1.0a4-Azurit
Parts:
- Dual1, Dual2: footprint ACS712:MC_33926_31polig_mit_Bohrloch_neue_Masse -> ACS712:MC_33926_31polig_mit_Bohrloch_neue_Masse_mit_zweite_Lochreihe
Changed lines of the file:
@@
 EESchema Schematic File Version 2
+LIBS:ardumower mega shield svn-cache
 LIBS:Wlan_ESP8266
 LIBS:power
-LIBS:ardumower mega shield svn-cache
+LIBS:conn
+LIBS:uln-udn
 EELAYER 25 0
 EELAYER END
@@
 F 0 "Dual1" H 3555 1335 60  0000 C CNN
 F 1 "MC33926" H 3575 3385 60  0000 C CNN
-F 2 "ACS712:MC_33926_31polig_mit_Bohrloch_neue_Masse" H 3755 2335 60  0001 C CNN
+F 2 "ACS712:MC_33926_31polig_mit_Bohrloch_neue_Masse_mit_zweite_Lochreihe" H 3755 2335 60  0001 C CNN
 F 3 "" H 3755 2335 60  0000 C CNN
 	1    3605 2285
@@
 pinMotorRightFault
 $Comp
-L GND #PWR0117
+L GND #PWR0123
 U 1 1 553D988C
 P 2415 1535
-F 0 "#PWR0117" H 2415 1285 60  0001 C CNN
+F 0 "#PWR0123" H 2415 1285 60  0001 C CNN
 F 1 "GND" V 2415 1310 60  0000 C CNN
 F 2 "" H 2415 1535 60  0000 C CNN
@@
 $EndComp
 $Comp
-L +5V #PWR0118
+L +5V #PWR0124
 U 1 1 553D98BA
 P 2415 1635
-F 0 "#PWR0118" H 2415 1485 60  0001 C CNN
+F 0 "#PWR0124" H 2415 1485 60  0001 C CNN
 F 1 "+5V" V 2415 1855 60  0000 C CNN
 F 2 "" H 2415 1635 60  0000 C CNN
@@
 pinMotorLeftFault
 $Comp
-L GND #PWR0119
+L GND #PWR0125
 U 1 1 553DA932
 P 2415 2435
-F 0 "#PWR0119" H 2415 2185 60  0001 C CNN
+F 0 "#PWR0125" H 2415 2185 60  0001 C CNN
 F 1 "GND" V 2415 2210 60  0000 C CNN
 F 2 "" H 2415 2435 60  0000 C CNN
@@
 $EndComp
 $Comp
-L +5V #PWR0120
+L +5V #PWR0126
 U 1 1 553DA938
 P 2415 2535
-F 0 "#PWR0120" H 2415 2385 60  0001 C CNN
+F 0 "#PWR0126" H 2415 2385 60  0001 C CNN
 F 1 "+5V" V 2415 2755 60  0000 C CNN
 F 2 "" H 2415 2535 60  0000 C CNN
@@
 pinMotorLeftDir
 $Comp
-L +5V #PWR0121
+L +5V #PWR0127
 U 1 1 553DB240
 P 1680 2835
-F 0 "#PWR0121" H 1680 2685 60  0001 C CNN
+F 0 "#PWR0127" H 1680 2685 60  0001 C CNN
 F 1 "+5V" V 1680 3055 60  0000 C CNN
 F 2 "" H 1680 2835 60  0000 C CNN
@@
 $EndComp
 $Comp
-L GND #PWR0122
+L GND #PWR0128
 U 1 1 553DB249
 P 2415 2935
-F 0 "#PWR0122" H 2415 2685 60  0001 C CNN
+F 0 "#PWR0128" H 2415 2685 60  0001 C CNN
 F 1 "GND" V 2415 2710 60  0000 C CNN
 F 2 "" H 2415 2935 60  0000 C CNN
@@
 F 0 "Dual2" H 3540 4585 60  0000 C CNN
 F 1 "MC33926" H 3560 6635 60  0000 C CNN
-F 2 "ACS712:MC_33926_31polig_mit_Bohrloch_neue_Masse" H 3740 5585 60  0001 C CNN
+F 2 "ACS712:MC_33926_31polig_mit_Bohrloch_neue_Masse_mit_zweite_Lochreihe" H 3740 5585 60  0001 C CNN
 F 3 "" H 3740 5585 60  0000 C CNN
 	1    3590 5535
@@
 pinMotorMowFault
 $Comp
-L GND #PWR0123
+L GND #PWR0129
 U 1 1 553DEB1E
 P 2400 4785
-F 0 "#PWR0123" H 2400 4535 60  0001 C CNN
+F 0 "#PWR0129" H 2400 4535 60  0001 C CNN
 F 1 "GND" V 2400 4560 60  0000 C CNN
 F 2 "" H 2400 4785 60  0000 C CNN
@@
 $EndComp
 $Comp
-L +5V #PWR0124
+L +5V #PWR0130
 U 1 1 553DEB24
 P 2400 4885
-F 0 "#PWR0124" H 2400 4735 60  0001 C CNN
+F 0 "#PWR0130" H 2400 4735 60  0001 C CNN
 F 1 "+5V" V 2400 5105 60  0000 C CNN
 F 2 "" H 2400 4885 60  0000 C CNN
@@
 pinMotorMowEnable
 $Comp
-L GND #PWR0125
+L GND #PWR0131
 U 1 1 553DEB38
 P 2400 5685
-F 0 "#PWR0125" H 2400 5435 60  0001 C CNN
+F 0 "#PWR0131" H 2400 5435 60  0001 C CNN
 F 1 "GND" V 2400 5460 60  0000 C CNN
 F 2 "" H 2400 5685 60  0000 C CNN
@@
 $EndComp
 $Comp
-L +5V #PWR0126
+L +5V #PWR0132
 U 1 1 553DEB3E
 P 2400 5785
-F 0 "#PWR0126" H 2400 5635 60  0001 C CNN
+F 0 "#PWR0132" H 2400 5635 60  0001 C CNN
 F 1 "+5V" V 2400 6005 60  0000 C CNN
 F 2 "" H 2400 5785 60  0000 C CNN
@@
 $EndComp
 $Comp
-L +5V #PWR0127
+L +5V #PWR0133
 U 1 1 553DEB4A
 P 1530 6085
-F 0 "#PWR0127" H 1530 5935 60  0001 C CNN
+F 0 "#PWR0133" H 1530 5935 60  0001 C CNN
 F 1 "+5V" V 1530 6305 60  0000 C CNN
 F 2 "" H 1530 6085 60  0000 C CNN
@@
 $EndComp
 $Comp
-L GND #PWR0128
+L GND #PWR0134
 U 1 1 553DEB51
 P 2400 6185
-F 0 "#PWR0128" H 2400 5935 60  0001 C CNN
+F 0 "#PWR0134" H 2400 5935 60  0001 C CNN
 F 1 "GND" V 2400 5960 60  0000 C CNN
 F 2 "" H 2400 6185 60  0000 C CNN
@@
 $EndComp
 $Comp
-L +24V #PWR0129
+L +24V #PWR0135
 U 1 1 553E3A94
 P 10435 910
-F 0 "#PWR0129" H 10435 760 60  0001 C CNN
+F 0 "#PWR0135" H 10435 760 60  0001 C CNN
 F 1 "+24V" H 10435 1050 60  0000 C CNN
 F 2 "" H 10435 910 60  0000 C CNN
@@
 $EndComp
 $Comp
-L GND #PWR0130
+L GND #PWR0136
 U 1 1 553E3A9A
 P 10435 1260
-F 0 "#PWR0130" H 10435 1010 60  0001 C CNN
+F 0 "#PWR0136" H 10435 1010 60  0001 C CNN
 F 1 "GND" H 10435 1110 60  0000 C CNN
 F 2 "" H 10435 1260 60  0000 C CNN
@@
 $EndComp
 $Comp
-L +24V #PWR0131
+L +24V #PWR0137
 U 1 1 553E4041
 P 10425 1845
-F 0 "#PWR0131" H 10425 1695 60  0001 C CNN
+F 0 "#PWR0137" H 10425 1695 60  0001 C CNN
 F 1 "+24V" H 10425 1985 60  0000 C CNN
 F 2 "" H 10425 1845 60  0000 C CNN
@@
 $EndComp
 $Comp
-L GND #PWR0132
+L GND #PWR0138
 U 1 1 553E4047
 P 10425 2195
-F 0 "#PWR0132" H 10425 1945 60  0001 C CNN
+F 0 "#PWR0138" H 10425 1945 60  0001 C CNN
 F 1 "GND" H 10425 2045 60  0000 C CNN
 F 2 "" H 10425 2195 60  0000 C CNN
@@
 $EndSheet
 $Bitmap
-Pos 9540 5630
+Pos 13325 5585
 Scale 2,000000
 Data
@@
 F8 F5 C7 F5 0E 3D 04 96 50 D8 96 35 42 9C E9 5A A7 8F FB 27 FF DC 2D EF 81 BD BF 1B 22 9B 87 00
 88 23 34 49 C4 FA FE 71 0F 3C 75 DF B2 7F C4 7E 07 9C 74 EA 29 98 AD 40 AA 86 14 64 89 65 C7 75
-85 53 4C B1 97 F1 FF 00 89 51 C8 4B C2 DC 5E A4 00 00 00 00 49 45 4E 44 AE 42 60 82 18
+85 53 4C B1 97 F1 FF 00 89 51 C8 4B C2 DC 5E A4 00 00 00 00 49 45 4E 44 AE 42 60 82 C7
 EndData
 $EndBitmap
 $Bitmap
-Pos 9120 4020
+Pos 13235 3985
 Scale 1,000000
 Data
@@
 94 6B 1D B7 0F 85 FF C6 86 DF 19 D7 CC C0 BB DD 16 35 D3 A5 4D 8D AC 19 82 D7 C8 C8 C8 C8 A8 10
 6D 93 08 99 F1 18 8C A6 4D 07 DE E0 44 58 CD 11 23 23 23 23 23 23 23 23 23 23 23 23 23 23 25 FD
-7F 58 5B 3B A6 13 40 A6 96 00 00 00 00 49 45 4E 44 AE 42 60 82 23
+7F 58 5B 3B A6 13 40 A6 96 00 00 00 00 49 45 4E 44 AE 42 60 82 A1
 EndData
 $EndBitmap
@@
 Connection ~ 1740 2835
 $Comp
-L GND #PWR0133
+L GND #PWR0139
 U 1 1 5558B071
 P 1740 3470
-F 0 "#PWR0133" H 1740 3220 60  0001 C CNN
+F 0 "#PWR0139" H 1740 3220 60  0001 C CNN
 F 1 "GND" V 1740 3245 60  0000 C CNN
 F 2 "" H 1740 3470 60  0000 C CNN
@@
 	1740 3470 1740 3380
 $Comp
-L GND #PWR0134
+L GND #PWR0140
 U 1 1 5558B77B
 P 1570 6795
-F 0 "#PWR0134" H 1570 6545 60  0001 C CNN
+F 0 "#PWR0140" H 1570 6545 60  0001 C CNN
 F 1 "GND" V 1570 6570 60  0000 C CNN
 F 2 "" H 1570 6795 60  0000 C CNN
@@
 $EndComp
 $Comp
-L GND #PWR0135
+L GND #PWR0141
 U 1 1 5558BA10
 P 1980 6795
-F 0 "#PWR0135" H 1980 6545 60  0001 C CNN
+F 0 "#PWR0141" H 1980 6545 60  0001 C CNN
 F 1 "GND" V 1980 6570 60  0000 C CNN
 F 2 "" H 1980 6795 60  0000 C CNN
@@
 $EndComp
 $Comp
-L GND #PWR0136
+L GND #PWR0142
 U 1 1 5558C056
 P 2195 3545
-F 0 "#PWR0136" H 2195 3295 60  0001 C CNN
+F 0 "#PWR0142" H 2195 3295 60  0001 C CNN
 F 1 "GND" V 2195 3320 60  0000 C CNN
 F 2 "" H 2195 3545 60  0000 C CNN
