File: pcb/megashield_svn_1.3_geoeffnet/Sonstiges.sch (KiCad schematic (older format))
At the start: 4 parts

Commit message: Import dernière version
1.0a4-Azurit
Parts:
- removed SP1: SPEAKER, ACS712:Buzzer_12x9.5RM7.6_RM5.0, symbol SPEAKER
Changed lines of the file:
@@
 EESchema Schematic File Version 2
+LIBS:ardumower mega shield svn-cache
 LIBS:Wlan_ESP8266
 LIBS:power
-LIBS:ardumower mega shield svn-cache
+LIBS:conn
+LIBS:uln-udn
 EELAYER 25 0
 EELAYER END
@@
 Comment4 ""
 $EndDescr
-$Comp
-L SPEAKER SP1
-U 1 1 55401981
-P 2165 1300
-F 0 "SP1" H 2065 1550 70  0000 C CNN
-F 1 "SPEAKER" H 2065 1050 70  0000 C CNN
-F 2 "ACS712:Buzzer_12x9.5RM7.6_RM5.0" H 2165 1300 60  0001 C CNN
-F 3 "" H 2165 1300 60  0000 C CNN
-F 4 "R: SUMMER TDB 05" H 2165 1300 60  0001 C CNN "Bestellnummer"
-	1    2165 1300
-	1    0    0    -1
-$EndComp
-$Comp
-L GND #PWR0153
-U 1 1 55401A25
-P 1615 1200
-F 0 "#PWR0153" H 1615 950 60  0001 C CNN
-F 1 "GND" V 1615 985 60  0000 C CNN
-F 2 "" H 1615 1200 60  0000 C CNN
-F 3 "" H 1615 1200 60  0000 C CNN
-	1    1615 1200
-	0    1    -1   0
-$EndComp
-Wire Wire Line
-	1865 1200 1615 1200
-Text GLabel 1615 1400 0    39   Input ~ 0
-pinBuzzer
-Wire Wire Line
-	1865 1400 1615 1400
 $Comp
 L JUMPER JP14
@@
 $EndComp
 $Comp
-L +3.3V #PWR0154
+L +3.3V #PWR0159
 U 1 1 553CB63B
 P 2775 2220
-F 0 "#PWR0154" H 2775 2180 30  0001 C CNN
+F 0 "#PWR0159" H 2775 2180 30  0001 C CNN
 F 1 "+3.3V" V 2775 2385 30  0000 C CNN
 F 2 "" H 2775 2220 60  0000 C CNN
@@
 $EndComp
 $Comp
-L +5V #PWR0155
+L +5V #PWR0160
 U 1 1 553CB667
 P 2770 2650
-F 0 "#PWR0155" H 2770 2500 60  0001 C CNN
+F 0 "#PWR0160" H 2770 2500 60  0001 C CNN
 F 1 "+5V" V 2770 2860 60  0000 C CNN
 F 2 "" H 2770 2650 60  0000 C CNN
