File: pcb/megashield_svn_1.3_geoeffnet/Stepdownwandler.sch (KiCad schematic (older format))
At the start: 18 parts, among them U1 DC 10V, U6 DC 3,3V, U7 DC 5V

Commit message: Import dernière version
1.0a4-Azurit
Parts:
- removed R24, R25, R26: 0, ACS712:Resistor_Horizontal_RM15mm, symbol R
- removed ZD1: ZD-5W 3,3V Optional, ACS712:Diode_ligend_RM10, symbol DIODE
- removed ZD2: ZD-5W 5,1 Optional, ACS712:Diode_ligend_RM10, symbol DIODE
- removed ZD3: ZD-5W 12V Optional, ACS712:Diode_ligend_RM10, symbol DIODE
- added DBY13, DBY14, DBY15, DBY16, DBY17, DBY18: BY 500/1000, ACS712:Diode_liegend_BY500_1000_RM15, symbol DIODE
- added DKE5, DKE6, DKE7: 15KE33CA, ACS712:Diode_15KE33CA, symbol 15KEXXC
- added PRFA6, PRFA7: PFRA 040, ACS712:PRFA_500_stehend, symbol F_10A
- added PRFA8: PFRA 040, symbol F_10A
- PRFA3, PRFA4, PRFA5: value PFRA 185 -> PFRA 040; Bestelllink http://www.reichelt.de/index.html?ACTION=3;ARTICLE=35184;SE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 -> https://www.reichelt.de/PFRA-040/3/index.html?&ACTION=3&LA=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; Bestellnummer R: PFRA 185 -> R: PFRA 040
Connections:
- net GND: now also DBY14.1 (A), DBY17.1 (A), DBY18.1 (A), DKE5.2, DKE6.2, DKE7.2
- net Stepdownwandler_24V_In: now also PRFA6.2, PRFA7.2, PRFA8.2; no longer U1.3 (VIN), U6.3 (VIN), U7.3 (VIN)
- net at PRFA3.2, U7.2 (Vout): now also DBY13.1 (A), DBY14.2 (K)
- net at PRFA5.2, U6.2 (Vout): now also DBY16.1 (A), DBY18.2 (K)
- net at PRFA4.2, U1.2 (Vout): now also DBY15.1 (A), DBY17.2 (K)
- new net: DBY13.2 (K), DKE5.1, PRFA6.1, U7.3 (VIN)
- new net: DBY16.2 (K), DKE7.1, PRFA8.1, U6.3 (VIN)
- new net: DBY15.2 (K), DKE6.1, PRFA7.1, U1.3 (VIN)
Other:
- note added: "Jürgen von 6.6.2015 \n3v 400ma eingang ausgang \n5v max 400ma eingang ausgang \n10v max 400ma eingang ausgang\n\nden 100µF ELKO kannst du durch einen 330nF Kerko ersetzen\ndie ELKOS setzen wir z.T an einer anderen Stelle im Board ein\nwo es mehr sinn macht das gehen wir nochmal an"
- note removed: "pfra Sicherung müssen von dem Wert her noch angepasst werden"
- moved on the sheet: C2, C7, C8, PRFA3, PRFA4, U1, U6, U7
