File: pcb/megashield_svn_1.3_geoeffnet/Stiftleisten.sch (KiCad schematic (older format))
At the start: 19 parts, among them P11 Bumper, P13 RC Remote, P14 Meas V, P19 Tilt sens, P32 Voltage header GND, P33 Voltage header 5V, P34 Voltage header 3,3V, P38 Status LEDs GND, P4 MowRpm, P40 UserSwitsch, P41 Rain, P48 Reset, P6 Lawn sens, P7 Status LEDs

Commit message: Import dernière version
1.0a4-Azurit
Parts:
- removed P38: Status LEDs GND, ACS712:Pin_Header_Straight_1x08, symbol CONN_01X08
- removed P7: Status LEDs, ACS712:Pin_Header_Straight_1x08, symbol CONN_01X08
- added IC1: UDN2981A, uln-udn-DIL18, symbol UDN2981A
- added P38: Status LEDs GND, symbol CONN_01X11
- added P7: Status LEDs, symbol CONN_01X11
- added R11: 1K5, ACS712:Resistor_Horizontal_RM10mm, symbol R
- added R20, R21, R24, R25, R26, R5: 220, ACS712:Resistor_Horizontal_RM10mm, symbol R
- added R41: 4,7K, ACS712:Resistor_Horizontal_RM10mm, symbol R
- added SP1: SPEAKER, ACS712:Buzzer_12x9.5RM7.6_RM5.0, symbol SPEAKER
- P4: Bestelllink (none) -> Value
Connections:
- net +5V: now also IC1.9 (VS), R41.2
- net DuoLED-Rot: now also IC1.2 (I2)
- net DuoLED_Grün: now also IC1.1 (I1)
- net GND: now also IC1.10 (GND), P38.1 (P1), P38.10 (P10), P38.11 (P11), P38.2 (P2), P38.3 (P3), P38.4 (P4), P38.5 (P5), P38.6 (P6), P38.7 (P7), P38.8 (P8), P38.9 (P9), P7.1 (P1), SP1.1
- net Led-Status: now also IC1.3 (I3)
- net StationLed: now also R11.1
- net pinMotorMowRpm: now also R41.1
- net LedPin-24v: no longer names the net of R2.2
- net LedPin-24v: now also P7.3 (P3)
- net LedPin-3V: no longer names the net of R23.2
- net LedPin-3V: now also P7.2 (P2)
- net LedPin-5v: no longer names the net of R1.2
- net LedPin-5v: now also P7.4 (P4)
- new net: P7.10 (P10), R26.2
- new net: P7.11 (P11), R25.2
- new net: P7.5 (P5), R11.2
- new net: P7.6 (P6), R21.2
- new net: P7.7 (P7), R20.2
- new net: P7.8 (P8), R5.2
- new net: P7.9 (P9), R24.2
- new net: IC1.11 (O8), SP1.2
- new net: IC1.16 (O3), R5.1
- new net: IC1.17 (O2), R20.1
- new net: IC1.18 (O1), R21.1
- new net: IC1.13 (O6), R25.1
- new net: IC1.14 (O5), R26.1
- new net: IC1.15 (O4), R24.1
- new net Led-BT: IC1.4 (I4)
- new net Led-Laderelais: IC1.6 (I6)
- new net Led-Wlan: IC1.5 (I5)
- new net pinBuzzer: IC1.8 (I8)
- no-connect marks 0 -> 2
Other:
- note added: "P7 und P38 (evl2) mal so anorden das vom Abstand\nher eine Led Leiste eingelötet werden kann.\n"
- note added: "bei den LEd müssen noch die Vorwiderstände bzw Transistoren eingebaut werden"
- moved on the sheet: R1, R2, R23
