File: pcb/megashield_svn_1.3_geoeffnet/ardumower mega shield svn.kicad_pcb (KiCad board)
At the start: 2 copper layers, 271.8 x 114.3 mm, 242 parts, among them K3 RELAY_2RT, P1 Sonar C., P10 GPS, P11 Bumper, P12 P.Left, P13 RC Remote, P14 Meas V, P15 Left, P16 V.OUT, P17 V.OUT, P18 Right, P19 Tilt sens, P2 Sonar R., P20 Button, P21 DropRight, P22 Res.AD6, P23 I2C Res.1, P24 I2C Res.2, P25 Res.Pin9, P26 Res.Pin4, P27 Res.Pin0, P28 Res.Pin8, P29 Res.Pin1, P3 Sonar L., P30 P.Right, P31 DropLeft, P32 Voltage header GND, P33 Voltage header 5V, P34 Voltage header 3,3V, P35 Resv.Pin49, P36 Res24V-2, P37 Mower, P38 Status LEDs GND, P39 Res24V-1, P4 MowRpm, P40 UserSwitsch, P41 Rain, P42 Charger connector, P43 Battery, P44 Wlan, P45 I2C Res.3, P46 I2C Res.4, P47 Not Aus, P48 Reset, P49 Res.AD10, P5 IMU Compas, P6 Lawn sens, P7 Status LEDs, P8 ODO Right, P9 ODO Left, Q1 BC547, Q2 IRF9530N, Q3 IRF9540N, Q4 BC337, Q5 IRF9530N, U1 DC 10V, U10 I2C_5-3V, U11 Wlan_ESP8266, U2 Bluetooth_CZ_HC_05, U3 INA169, U6 DC 3,3V, U7 DC 5V, U8 DS1307+

Commit message: Import dernière version
1.0a4-Azurit
Parts:
- removed CC20, CC5: 100nF, Capacitors_ThroughHole:C_Disc_D3_P2.5
- removed D8: BlueLED, ACS712:Diode_LED_5mm_round_vertical
- added R41: 4,7K, ACS712:Resistor_Horizontal_RM10mm, F.Cu at (205.5, 43.2)
- CC1: value 100 nF -> 100nF
- CC40, CC6: moved to B.Cu
- Dual1, Dual2: footprint ACS712:MC_33926_31polig_mit_Bohrloch_neue_Masse -> ACS712:MC_33926_31polig_mit_Bohrloch_neue_Masse_mit_zweite_Lochreihe
- P38, P7: footprint ACS712:Pin_Header_Straight_1x08 -> ACS712:Pin_Header_Straight_1x09
- RP1, RP2: value 150 -> 220R
- RR1, RR2: value C0,1uF -> (0,01uF) 10nF
- moved JP12 2.54 mm to (114.3, 50.8)
- moved JP13 2.54 mm to (119.4, 50.8)
- moved JP15 2.54 mm to (124.5, 50.8)
- moved JP9 2.54 mm to (109.2, 50.8)
- moved JP14 2.54 mm to (121.9, 50.8)
- moved JP16 2.54 mm to (127.0, 50.8)
- moved JP2 2.54 mm to (106.7, 50.8)
- moved JP3 2.54 mm to (116.8, 50.8)
- moved JP8 2.54 mm to (111.8, 50.8)
- moved KE4 2.26 mm to (256.0, 50.4)
- moved KE3 1.09 mm to (255.5, 98.6)
- moved R39 0.89 mm to (186.7, 50.7)
- moved CC32 0.13 mm to (216.5, 66.3)
- moved CC16 0.13 mm to (179.1, 132.1)
Connections:
- R22 pad 2: Net-(D8-Pad2) -> Led-BT
Routing:
- net Led-BT: track 0.00 -> 102.1 mm, vias 0 -> 4
- net pinMotorMowRpm: track 28.3 -> 58.0 mm, vias 1 -> 2
- net Net-(D8-Pad2): track 20.7 -> 0.00 mm, vias 2 -> 0
- net PowerA3,3: track 50.1 -> 68.7 mm
- net pinBatteryVoltage: track 21.5 -> 11.6 mm, vias 2 -> 1
- net Net-(Dual2-Pad9): track 112.7 -> 120.3 mm, vias 5 -> 4
- net /Motortreiber/Dual1_Ms_Rechts/MotorRechtsA: track 33.3 -> 40.6 mm
- net pinChargeVoltage: track 15.1 -> 9.27 mm
- net pinMotorRightSense: track 115.6 -> 110.3 mm
- net /Motortreiber/Dual2_Ms_Mower/MotorMowerA: track 42.8 -> 47.9 mm, vias 2 -> 3
- net ReserveAD6: track 46.1 -> 50.2 mm
- net LedPin-3V: track 43.0 -> 47.0 mm
- net GND: track 1982.2 -> 1979.2 mm
- net Net-(JP2-Pad2): track 42.0 -> 39.5 mm
- net /Motortreiber/Dual1_Ms_Rechts/MotorRechtsB: track 46.0 -> 48.5 mm, vias 3 -> 4
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Other:
- board text added: "LED BT"
