File: pcb/megashield_svn_1.3_geoeffnet/ardumower mega shield svn.sch (KiCad schematic (older format))
At the start: 33 parts, among them K3 RELAY_2RT, P42 Charger connector, P43 Battery, P47 Not Aus, Q1 BC547, U3 INA169

Commit message: Import dernière version
1.0a4-Azurit
Parts:
- removed R11: 1K5, ACS712:Resistor_Horizontal_RM10mm, symbol R
- removed R20, R21, R5: 220R, ACS712:Resistor_Horizontal_RM10mm, symbol R
- added CC5: 100nf, symbol Kondensator
- added D1, D12, D2, D3: MBR 1045, ACS712:MBR1045, symbol DIODE
- added D4, D7, D8, D9: 1N4148, ACS712:Diode_ligend_RM10, symbol DIODE
- CC1: value 100 nF -> 100nF
- RP1, RP2: value 150 -> 220R
- RR1, RR2: value C0,1uF -> (0,01uF) 10nF
- renumbered KE1 to DKE1, KE2 to DKE2
Connections:
- net Batteriespannung/Batteriespannung: now also D9.2 (K); no longer DKE1.2, K3.1 (T1), P47.1 (P1)
- net DuoLED-Rot: now also SHIELD1.7
- net DuoLED_Grün: now also SHIELD1.6
- net GND: now also CC5.2, D1.1 (A), D2.1 (A), D4.2 (K); no longer Q1.E
- net Ladespannung/Ladespannung: now also D7.2 (K); no longer EF1.1
- net Led-Status: now also SHIELD1.13
- net StationLed: now also D8.2 (K)
- net UnterSpannungsSchutz/Batterieeingang 24V: now also D12.2 (K), D3.2 (K)
- net Verpols.L/Verpols.L.aus: no longer K3.16 (T2), R19.1
- net at SHIELD1.AREF: now also CC5.1
- net at D11.1 (A): now also EF1.1, K3.16 (T2), D1.2 (K), D12.1 (A), D7.1 (A), D8.1 (A); no longer R19.2
- net pinChargingEnable renamed Led-Laderelais
- new net: D2.2 (K), D3.1 (A), D9.1 (A), DKE1.2, K3.1 (T1), P47.1 (P1)
- new net: D4.1 (A), Q1.E
- no-connect marks 9 -> 6
Other:
- note added: "25052015 Kondesatornetzwerk wert geändert 100nf - Jürgen\n25052015 Odemetrie 4 Widerstände 4,7k eingefügt\n25052015 Widerstansnetzwerk Wert geändert von 150 Ohm nach 220 Ohm - Jürgen\n25052015 Footprint MC Driver geändert\n28052015 MowRpm 4,7K Widerstand eingefügt\n20150603 AREF Kondesator eingefügt"
- note added: "Bei den Schutzdioden noch den den Drahtdurchmesser und Lochdruchmesser im Footprint kontrollieren.\nBe den Kidioden das Loch für den footprint von 1mm auf 1,2mm vergrößert"
- note added: "Schutzdiode (Angstdiode)Transistor\nfür den Fall das die Ladespannung verpolt ist"
- note added: "Verpolschutz\nAlternativ"
- note added: "zu den Motortreibern"
- moved on the sheet: D11, DKE1, R19
