File: pcb/megashield_svn_1.3_geoeffnet/serielle Schnittstelle.sch (KiCad schematic (older format))
At the start: 16 parts, among them P10 GPS, P44 Wlan, U11 Wlan_ESP8266, U2 Bluetooth_CZ_HC_05

Commit message: Import dernière version
1.0a4-Azurit
Parts:
- removed D8: BlueLED, ACS712:Diode_LED_5mm_round_vertical, symbol CONN_2
- added JP4: Wlan, ACS712:Pin_Header_Straight_1x02, symbol JUMPER
Connections:
- net GND: now also JP4.2
- net Led-BT: now reaches R22.2
- net at U11.GP_0 (GP_IO0): now also JP4.1
- net Led-Wlan: now reaches U11.GP_2 (GP_IO2)
- no-connect marks 3 -> 1
Other:
- note added: "https://github.com/FredericG-BE/ardumower/wiki/Using-ESP8266-WIFI-module-on-Ardumower\nBy adding a LED, it is easy to see the state of the ESP8266 firmware: \nconnecting to the WIFI Access Point, Connected, PFOD connected,\n ... Also here, perhaps a LED and resistor could be added directly to the ESP8266 PCB.\nObserve that the GIO bins can only source 12mA.\n I used a 220 Ohm resistor, which will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"
- moved on the sheet: P10, U11
